File: hardware/Revision A1/mcore-h616-breakout-RevA1.brd (EAGLE design)
At the start: 88 x 74.5 mm, 62 parts, among them CON1 C136421 - HDMI-519, CON4 LPJG0926HENL, IC1 LD1117-3.3, SW1 SPNO

Commit message: clean-up and mfg release for rev A1
Parts:
- removed R22, R23, R24: 49.9Ω, ok-discretes-dev:_PKG_R_0402
- removed TP6: TP, ok-testdebug-dev:TP_DOT_1.5X1.5MM
- removed U$1: C111196 - TF-15x15, ok-connectors-dev:TF/SHENZHEN-SPECIAL
- added J5: (no value), SparkFun-Connectors:1X02_LOCK
- added R18: 100, ok-discretes-dev:_PKG_R_0402
- added R19: 10k, ok-discretes-dev:_PKG_R_0402
- added R2: 5k1, ok-discretes-dev:_PKG_R_0402
- added TP4: TP, ok-testdebug-dev:TP_DOT_1.5X1.5MM
- C1: value 10n -> 47u; device ok-discretes-dev:_PKG_C_0402 -> ok-discretes-dev:_PKG_C_1206
- C10, C8: value 100n -> 47u; device ok-discretes-dev:_PKG_C_0402 -> ok-discretes-dev:_PKG_C_1206
- C3, C4, C7: value 10u -> 47u
- C5: value 10u -> 10n; device ok-discretes-dev:_PKG_C_1206 -> ok-discretes-dev:_PKG_C_0402
- C6, C9: value 10u -> 100n; device ok-discretes-dev:_PKG_C_1206 -> ok-discretes-dev:_PKG_C_0402
- CON1: value C136421 - HDMI-519 -> (none); device Wurth_Connectors_WR-HDMI:685119136923 -> ok-connectors-dev:JING_912-121A2023S10100
- CON3: device ok-connectors-dev:CON_2.54MM_TH_2X20 -> ok-connectors-dev:USBC_C-31-M-12
- CON4: value LPJG0926HENL -> C136421 - HDMI-519; device ok-connectors-dev:LPJG0926HENL -> Wurth_Connectors_WR-HDMI:685119136923
- CON5: value (none) -> LPJG0926HENL; device ok-connectors-dev:USBC_C-31-M-12 -> ok-connectors-dev:LPJG0926HENL
- CON6: value (none) -> C111196 - TF-15x15; device ok-connectors-dev:JING_912-121A2023S10100 -> ok-connectors-dev:TF/SHENZHEN-SPECIAL
- D3, D4: value C154821 -> RB520S30T1G
- J1: device SparkFun-Connectors:1X02_LOCK -> SparkFun-Connectors:1X04_LOCK
- J2: device SparkFun-Connectors:1X02_LOCK -> SparkFun-Connectors:1X03_LOCK
- J3: device SparkFun-Connectors:1X03_LOCK -> SparkFun-Connectors:1X02_LOCK
- J4: device SparkFun-Connectors:1X04_LOCK -> ok-connectors-dev:CON_2.54MM_TH_2X20
- R1: value 100 -> 5k1
- R13: value 100 -> 49.9Ω
- R14: value 1k -> 49.9Ω
- R15: value 470 -> 49.9Ω
- R16: value 10k -> 49.9Ω
- R17: value 27k 1% -> 10k
- R20: value 470 -> 100
- R21: value 49.9Ω -> 100
- R3: value 10k -> 100
- R6: value 5k1 -> 1k
- R7: value 5k1 -> 27k 1%
- R8: value 33 -> 100
- moved J3 89.9 mm to (73.6, 4.12), turned to 180 degrees
- moved CON6 78.3 mm to (80.6, 44.5), turned to 270 degrees
- moved R1 62.9 mm to (34.0, 10.8), turned to 0 degrees
- moved R3 60.9 mm to (70.6, 61.9), turned to 180 degrees
- moved R4 58.5 mm to (10.6, 51.6), turned to 0 degrees
- moved CON3 57.2 mm to (39.0, 4.70)
- moved R16 56.5 mm to (62.8, 24.9), turned to 90 degrees
- moved R5 55.8 mm to (13.0, 51.6), turned to 0 degrees
- moved CON1 55.0 mm to (5.30, 23.0), turned to 90 degrees
- moved J4 50.7 mm to (32.5, 61.5), turned to 0 degrees
- moved C5 46.1 mm to (50.0, 3.00), turned to 90 degrees
- moved J1 43.5 mm to (30.6, 10.9), turned to 270 degrees
- moved TP1 43.0 mm to (30.4, 71.1)
- moved CON5 43.0 mm to (77.3, 24.1), turned to 90 degrees
- moved TP2 42.5 mm to (20.9, 29.0), turned to 270 degrees
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- renumbered CON7 to CON2, CON8 to J6
Connections:
- net 5V: now also C1.2, C4.2, CON1.VBUS, D2.5, D4.2, J5.2; no longer C10.2, C5.2, CON6.VBUS, D1.5, D3.2, J2.2
- net GND: now also CON1.GND, CON1.P$5, CON1.P$6, CON3.GND@1, CON3.GND@2, CON3.P$1, CON3.P$2, CON3.P$3, CON3.P$4, CON3.P$5, CON3.P$7, CON3.P$8, CON4.1, CON4.10, CON4.13, CON4.4, CON4.7, CON4.SHELL, CON4.SHELL1, CON4.SHELL2, CON4.SHELL3, CON5.MH3, CON5.MH4, CON6.6, CON6.S1, CON6.S2, CON6.S3, CON6.S4, J2.1, J4.P$14, J4.P$20, J4.P$25, J4.P$30, J4.P$34, J4.P$39, J4.P$6, J4.P$9, R1.1, R2.1, TP1.TP, TP2.TP; no longer CON1.1, CON1.10, CON1.13, CON1.4, CON1.7, CON1.SHELL, CON1.SHELL1, CON1.SHELL2, CON1.SHELL3, CON3.P$14, CON3.P$20, CON3.P$25, CON3.P$30, CON3.P$34, CON3.P$39, CON3.P$9, CON4.MH3, CON4.MH4, CON5.GND@1, CON5.GND@2, CON5.P$1, CON5.P$2, CON5.P$3, CON5.P$4, CON5.P$5, CON5.P$6, CON5.P$7, CON5.P$8, CON6.GND, CON6.P$5, CON6.P$6, J4.1, R6.1, R7.1, TP3.TP, TP6.TP, U$1.6, U$1.S1, U$1.S2, U$1.S3, U$1.S4
- net H5V: now also CON4.18, D4.1; no longer CON1.18, D3.1
- net HCEC: now also R8.2; no longer R13.2
- net HDCEC: now also CON4.14, R7.1, R8.1; no longer CON1.14, R13.1, R17.1
- net HDHPD: now also CON4.19, R6.1; no longer CON1.19, R14.1
- net HDSCL: now also CON4.15; no longer CON1.15
- net HDSDA: now also CON4.16; no longer CON1.16
- net HHPD: now also C11.2, R6.2; no longer C16.2, R14.2
- net HTX0_N: now also CON4.9; no longer CON1.9
- net HTX0_P: now also CON4.8; no longer CON1.8
- net HTX1_N: now also CON4.6; no longer CON1.6
- net HTX1_P: now also CON4.5; no longer CON1.5
- net HTX2_N: now also CON4.3; no longer CON1.3
- net HTX2_P: now also CON4.2; no longer CON1.2
- net HTXC_N: now also CON4.12; no longer CON1.12
- net HTXC_P: now also CON4.11; no longer CON1.11
- net LAN_LED_G: now also R20.2; no longer R15.2
- net LAN_LED_Y: now also R21.2; no longer R20.2
- net LINEOUT_L: now also J1.3; no longer J4.3
- net LINEOUT_R: now also J1.4; no longer J4.4
- net LRADC: now also J1.2; no longer J4.2
- net N$1: now also R3.1; no longer R1.1
- net N$10: now also CON3.CC2, R1.2; no longer CON5.CC2, R6.2
- net N$2: now also CON5.16, R20.1; no longer CON4.16, R15.1
- net N$3: now also C14.2, CON5.4; no longer C15.2, CON4.4
- net N$30: now also C12.2, R13.1, R14.1; no longer C13.2, R21.1, R22.1
- net N$31: now also C13.2, R15.1, R16.1; no longer C12.2, R23.1, R24.1
- net N$4: now also C16.2, CON5.5; no longer C14.2, CON4.5
- net N$5: now also J4.P$2, J4.P$4, J5.1; no longer CON3.P$2, CON3.P$4, J2.1
- net N$6: now also CON5.18, R21.1; no longer CON4.18, R20.1
- net N$7: now also D3.1, R7.2; no longer D4.1, R17.2
- net N$9: now also CON3.CC1, R2.2; no longer CON5.CC1, R7.2
- net PH0/UART0-TX: now also J2.2, J4.P$8; no longer CON3.P$8, J3.2
- net PH1/UART0-RX: now also J2.3, J4.P$10; no longer CON3.P$10, J3.3
- net PH10: now also J4.P$36, MOD1.46; no longer CON3.P$36
- net PH2/UART5-TX: now also J4.P$11; no longer CON3.P$11
- net PH3/UART5-RX: now also J4.P$13; no longer CON3.P$13
- net PH4: now also J4.P$18; no longer CON3.P$18
- net PI0/I2S0-MCLK: now also J4.P$7; no longer CON3.P$7
- net PI1/I2S0-BCLK: now also J4.P$12; no longer CON3.P$12
- net PI10/TWI2-SDA: now also J4.P$27; no longer CON3.P$27
- net PI11: now also J4.P$29; no longer CON3.P$29
- net PI12: now also J4.P$31; no longer CON3.P$31
- net PI13/UART4-TX/PWM3: now also J4.P$15; no longer CON3.P$15
- net PI14/UART4-RX/PWM4: now also J4.P$16; no longer CON3.P$16
- net PI15: now also J4.P$33; no longer CON3.P$33
- net PI16: now also J4.P$37; no longer CON3.P$37
- net PI2/I2S0-LRCK: now also J4.P$35; no longer CON3.P$35
- net PI3/I2S0-DIN: now also J4.P$40; no longer CON3.P$40
- net PI4/I2S0-DOUT: now also J4.P$38; no longer CON3.P$38
- net PI5/UART2-TX: now also J4.P$32; no longer CON3.P$32
- net PI6/UART2-RX: now also J4.P$22; no longer CON3.P$22
- net PI7/TWI1-SCK: now also J4.P$5, R5.2; no longer CON3.P$5, R16.2
- net PI8/TWI1-SDA: now also J4.P$3, R4.2; no longer CON3.P$3, R3.2
- net PI9/TWI2-SCK: now also J4.P$28; no longer CON3.P$28
- net RXI_N: now also CON5.6, R16.2; no longer CON4.6, R24.2
- net RXI_P: now also CON5.3, R15.2; no longer CON4.3, R23.2
- net SCD0-CLK: now also R18.2; no longer R8.2
- net SCD0-CLK': now also CON6.5, R18.1; no longer R8.1, U$1.5
- net SCD0-CMD: now also CON6.3, R17.1; no longer R4.1, U$1.3
- net SCD0-D0: now also CON6.7; no longer U$1.7
- net SCD0-D1: now also CON6.8; no longer U$1.8
- net SCD0-D2: now also CON6.1; no longer U$1.1
- net SCD0-D3: now also CON6.2; no longer U$1.2
- net SCD0-DET: now also CON6.9, R19.1, TP4.TP; no longer R5.1, TP1.TP, U$1.9
- net SPI1-CLK: now also J4.P$23; no longer CON3.P$23
- net SPI1-CS0: now also J4.P$24; no longer CON3.P$24
- net SPI1-CS1: now also J4.P$26; no longer CON3.P$26
- net SPI1-MISO: now also J4.P$21; no longer CON3.P$21
- net SPI1-MOSI: now also J4.P$19; no longer CON3.P$19
- net TR0_TAP: now also CON5.11; no longer CON4.11
- net TR1_TAP: now also CON5.12; no longer CON4.12
- net TR2_TAP: now also CON5.13; no longer CON4.13
- net TR3_TAP: now also CON5.14; no longer CON4.14
- net TXO_N: now also CON5.2, R14.2; no longer CON4.2, R22.2
- net TXO_P: now also CON5.1, R13.2; no longer CON4.1, R21.2
- net USB0_N: now also CON3.DN1, CON3.DN2, D1.3; no longer CON5.DN1, CON5.DN2, D2.3
- net USB0_P: now also CON3.DP1, CON3.DP2, D1.1; no longer CON5.DP1, CON5.DP2, D2.1
- net USB1_N: now also CON1.DM, D2.4; no longer CON6.DM, D1.4
- net USB1_P: now also CON1.DP, D2.6; no longer CON6.DP, D1.6
- net USB2_N: now also D2.1; no longer D1.1
- net USB2_P: now also D2.3; no longer D1.3
- net VCC: now also C10.2, C15.2, CON5.15, CON5.17, CON6.4, D3.2, J4.P$1, J4.P$17, R17.2, R19.2, R3.2, R4.1, R5.1, TP3.TP; no longer C11.2, C4.2, CON3.P$1, CON3.P$17, CON4.15, CON4.17, D4.2, R1.2, R16.1, R3.1, R4.2, R5.2, TP2.TP, U$1.4
- net VUSB_IN: now also C5.2, CON3.VBUS@1, CON3.VBUS@2, D1.5, J3.2; no longer C1.2, CON5.VBUS@1, CON5.VBUS@2, D2.5, J1.2
Routing:
- net PH10: track 0.00 -> 52.1 mm, vias 0 -> 1
- net PI4/I2S0-DOUT: track 35.7 -> 38.4 mm
- net PI6/UART2-RX: track 25.4 -> 26.1 mm
- net PI16: track 43.6 -> 44.3 mm
- net GND: vias 267 -> 274
Other:
- board text added: "I2S0-LRCK"
- board text added: "I2S0-MCLK"
- board text added: "PH2"
- board text added: "PH3"
- board text added: "PI0"
- board text added: "PI10"
- board text added: "PI3/PWM3"
- board text added: "PI7"
- board text added: "PI8"
- board text added: "UART4-TX"
- board text added: "UART5-RX"
- board text added: "UART5-TX"
- board text removed: "5V In"
- board text removed: "aa"
- board text removed: "aaaa"
