File: hardware/Revision A1/mcore-h616-breakout-RevA1.sch (EAGLE design)
At the start: 62 parts, among them CON1 C136421 - HDMI-519, CON4 LPJG0926HENL, IC1 LD1117-3.3, SW1 SPNO

Commit message: clean-up and mfg release for rev A1
Parts:
- removed R22, R23, R24: 49.9Ω, ok-discretes-dev:RES-0402
- removed TP6: TP, ok-testdebug-dev:TP
- removed U$1: C111196 - TF-15x15, ok-connectors-dev:TF/SHENZHEN-SPECIAL
- added J5: (no value), SparkFun-Connectors:CONN_02LOCK
- added R18: 100, ok-discretes-dev:RES-0402
- added R19: 10k, ok-discretes-dev:RES-0402
- added R2: 5k1, ok-discretes-dev:RES-0402
- added TP4: TP, ok-testdebug-dev:TP
- C1: value 10n -> 47u; device ok-discretes-dev:CAP-0402 -> ok-discretes-dev:CAP-1206; JLCASSY C15195 -> C96123
- C10, C8: value 100n -> 47u; device ok-discretes-dev:CAP-0402 -> ok-discretes-dev:CAP-1206; JLCASSY C307331 -> C96123
- C12, C13, C14, C15: JLCASSY (none) -> C307331
- C3, C4, C7: value 10u -> 47u; JLCASSY C19702 -> C96123
- C5: value 10u -> 10n; device ok-discretes-dev:CAP-1206 -> ok-discretes-dev:CAP-0402; JLCASSY C19702 -> C15195
- C6, C9: value 10u -> 100n; device ok-discretes-dev:CAP-1206 -> ok-discretes-dev:CAP-0402; JLCASSY C19702 -> C307331
- CON1: value C136421 - HDMI-519 -> (none); device Wurth_Connectors_WR-HDMI:685119136923 -> ok-connectors-dev:USB-A-FEMALE-JING-912-121A2023S10100; JLCASSY (none) -> C42428
- CON2: JLCASSY (none) -> C42428
- CON3: device ok-connectors-dev:CON_2.54MM_TH_2X20 -> ok-connectors-dev:USBC_USB-C-12; JLCASSY (none) -> C165948
- CON4: value LPJG0926HENL -> C136421 - HDMI-519; device ok-connectors-dev:RJ45_POE_LPJG0926HENL -> Wurth_Connectors_WR-HDMI:685119136923; JLCASSY (none) -> C136421
- CON5: value (none) -> LPJG0926HENL; device ok-connectors-dev:USBC_USB-C-12 -> ok-connectors-dev:RJ45_POE_LPJG0926HENL
- CON6: value (none) -> C111196 - TF-15x15; device ok-connectors-dev:USB-A-FEMALE-JING-912-121A2023S10100 -> ok-connectors-dev:TF/SHENZHEN-SPECIAL; JLCASSY (none) -> C111196
- D3, D4: value C154821 -> RB520S30T1G; JLCASSY (none) -> C154821
- J1: device SparkFun-Connectors:CONN_02LOCK -> SparkFun-Connectors:CONN_04LOCK
- J2: device SparkFun-Connectors:CONN_02LOCK -> SparkFun-Connectors:CONN_03LOCK
- J3: device SparkFun-Connectors:CONN_03LOCK -> SparkFun-Connectors:CONN_02LOCK
- J4: device SparkFun-Connectors:CONN_04LOCK -> ok-connectors-dev:CON_2.54MM_TH_2X20
- L1: JLCASSY C1017 -> C75661
- R1: value 100 -> 5k1; JLCASSY C25076 -> C25905
- R10, R9: JLCASSY (none) -> C25871
- R11, R12: JLCASSY (none) -> C25076
- R13: value 100 -> 49.9Ω; JLCASSY (none) -> C25120
- R14: value 1k -> 49.9Ω; JLCASSY (none) -> C25120
- R15: value 470 -> 49.9Ω; JLCASSY (none) -> C25120
- R16: value 10k -> 49.9Ω; JLCASSY (none) -> C25120
- R17: value 27k 1% -> 10k; JLCASSY (none) -> C25744
- R20: value 470 -> 100; JLCASSY (none) -> C25076
- R21: value 49.9Ω -> 100; JLCASSY (none) -> C25076
- R3: value 10k -> 100; JLCASSY (none) -> C25076
- R6: value 5k1 -> 1k; JLCASSY (none) -> C11702
- R7: value 5k1 -> 27k 1%; JLCASSY (none) -> C25771
- R8: value 33 -> 100; JLCASSY C25744 -> C25076
- renumbered CON7 to CON2, CON8 to J6
Connections:
- net 5V: now also C1.2, C4.2, CON1.V, D2.REF, D4.A, J5.2; no longer C10.2, C5.2, CON6.V, D1.REF, D3.A, J2.2
- net GND: now also CON1.G, CON1.SHIELD1, CON1.SHIELD2, CON3.CHASSIS, CON3.GND, CON4.DDC/CECGROUND/HEACSHIELD, CON4.SHIELD, CON4.TMDSCLOCKSHIELD, CON4.TMDSDATA0SHIELD, CON4.TMDSDATA1SHIELD, CON4.TMDSDATA2SHIELD, CON5.MH3, CON5.MH4, CON6.GND, CON6.S1, CON6.S2, CON6.S3, CON6.S4, J2.1, J4.14, J4.20, J4.25, J4.30, J4.34, J4.39, J4.6, J4.9, R1.1, R2.1, TP1.TP, TP2.TP; no longer CON1.DDC/CECGROUND/HEACSHIELD, CON1.SHIELD, CON1.TMDSCLOCKSHIELD, CON1.TMDSDATA0SHIELD, CON1.TMDSDATA1SHIELD, CON1.TMDSDATA2SHIELD, CON3.14, CON3.20, CON3.25, CON3.30, CON3.34, CON3.39, CON3.6, CON3.9, CON4.MH3, CON4.MH4, CON5.CHASSIS, CON5.GND, CON6.G, CON6.SHIELD1, CON6.SHIELD2, J4.1, R6.1, R7.1, TP3.TP, TP6.TP, U$1.GND, U$1.S1, U$1.S2, U$1.S3, U$1.S4
- net H5V: now also CON4.+5VPOWER, D4.C; no longer CON1.+5VPOWER, D3.C
- net HCEC: now also R8.2; no longer R13.2
- net HDCEC: now also CON4.CEC, R7.1, R8.1; no longer CON1.CEC, R13.1, R17.1
- net HDHPD: now also CON4.HOTPLUGDETECT/HEAC-, R6.1; no longer CON1.HOTPLUGDETECT/HEAC-, R14.1
- net HDSCL: now also CON4.SCL; no longer CON1.SCL
- net HDSDA: now also CON4.SDA; no longer CON1.SDA
- net HHPD: now also C11.2, R6.2; no longer C16.2, R14.2
- net HTX0_N: now also CON4.TMDSDATA0-; no longer CON1.TMDSDATA0-
- net HTX0_P: now also CON4.TMDSDATA0+; no longer CON1.TMDSDATA0+
- net HTX1_N: now also CON4.TMDSDATA1-; no longer CON1.TMDSDATA1-
- net HTX1_P: now also CON4.TMDSDATA1+; no longer CON1.TMDSDATA1+
- net HTX2_N: now also CON4.TMDSDATA2-; no longer CON1.TMDSDATA2-
- net HTX2_P: now also CON4.TMDSDATA2+; no longer CON1.TMDSDATA2+
- net HTXC_N: now also CON4.TMDSCLOCK-; no longer CON1.TMDSCLOCK-
- net HTXC_P: now also CON4.TMDSCLOCK+; no longer CON1.TMDSCLOCK+
- net LAN_LED_G: now also R20.2; no longer R15.2
- net LAN_LED_Y: now also R21.2; no longer R20.2
- net LINEOUT_L: now also J1.3; no longer J4.3
- net LINEOUT_R: now also J1.4; no longer J4.4
- net LRADC: now also J1.2; no longer J4.2
- net N$1: now also R3.1; no longer R1.1
- net N$10: now also CON3.CC2, R1.2; no longer CON5.CC2, R6.2
- net N$2: now also CON5.K_GREEN, R20.1; no longer CON4.K_GREEN, R15.1
- net N$3: now also C14.2, CON5.TD2-@4; no longer C15.2, CON4.TD2-@4
- net N$30: now also C12.2, R13.1, R14.1; no longer C13.2, R21.1, R22.1
- net N$31: now also C13.2, R15.1, R16.1; no longer C12.2, R23.1, R24.1
- net N$4: now also C16.2, CON5.TD2-@5; no longer C14.2, CON4.TD2-@5
- net N$5: now also J4.2, J4.4, J5.1; no longer CON3.2, CON3.4, J2.1
- net N$6: now also CON5.K_YELLOW, R21.1; no longer CON4.K_YELLOW, R20.1
- net N$7: now also D3.C, R7.2; no longer D4.C, R17.2
- net N$9: now also CON3.CC1, R2.2; no longer CON5.CC1, R7.2
- net PH0/UART0-TX: now also J2.2, J4.8; no longer CON3.8, J3.2
- net PH1/UART0-RX: now also J2.3, J4.10; no longer CON3.10, J3.3
- net PH10: now also J4.36, MOD1.PH10/IR_RX/TCON_TRIG1/PH_EINT10; no longer CON3.36
- net PH2/UART5-TX: now also J4.11; no longer CON3.11
- net PH3/UART5-RX: now also J4.13; no longer CON3.13
- net PH4: now also J4.18; no longer CON3.18
- net PI0/I2S0-MCLK: now also J4.7; no longer CON3.7
- net PI1/I2S0-BCLK: now also J4.12; no longer CON3.12
- net PI10/TWI2-SDA: now also J4.27; no longer CON3.27
- net PI11: now also J4.29; no longer CON3.29
- net PI12: now also J4.31; no longer CON3.31
- net PI13/UART4-TX/PWM3: now also J4.15; no longer CON3.15
- net PI14/UART4-RX/PWM4: now also J4.16; no longer CON3.16
- net PI15: now also J4.33; no longer CON3.33
- net PI16: now also J4.37; no longer CON3.37
- net PI2/I2S0-LRCK: now also J4.35; no longer CON3.35
- net PI3/I2S0-DIN: now also J4.40; no longer CON3.40
- net PI4/I2S0-DOUT: now also J4.38; no longer CON3.38
- net PI5/UART2-TX: now also J4.32; no longer CON3.32
- net PI6/UART2-RX: now also J4.22; no longer CON3.22
- net PI7/TWI1-SCK: now also J4.5, R5.2; no longer CON3.5, R16.2
- net PI8/TWI1-SDA: now also J4.3, R4.2; no longer CON3.3, R3.2
- net PI9/TWI2-SCK: now also J4.28; no longer CON3.28
- net RXI_N: now also CON5.TD2-@6, R16.2; no longer CON4.TD2-@6, R24.2
- net RXI_P: now also CON5.TD2+, R15.2; no longer CON4.TD2+, R23.2
- net SCD0-CLK: now also R18.2; no longer R8.2
- net SCD0-CLK': now also CON6.CLK/SCLK, R18.1; no longer R8.1, U$1.CLK/SCLK
- net SCD0-CMD: now also CON6.CMD/DI, R17.1; no longer R4.1, U$1.CMD/DI
- net SCD0-D0: now also CON6.DAT0/D0; no longer U$1.DAT0/D0
- net SCD0-D1: now also CON6.DAT1; no longer U$1.DAT1
- net SCD0-D2: now also CON6.DAT2; no longer U$1.DAT2
- net SCD0-D3: now also CON6.DAT3/CS; no longer U$1.DAT3/CS
- net SCD0-DET: now also CON6.CD_SW, R19.1, TP4.TP; no longer R5.1, TP1.TP, U$1.CD_SW
- net SPI1-CLK: now also J4.23; no longer CON3.23
- net SPI1-CS0: now also J4.24; no longer CON3.24
- net SPI1-CS1: now also J4.26; no longer CON3.26
- net SPI1-MISO: now also J4.21; no longer CON3.21
- net SPI1-MOSI: now also J4.19; no longer CON3.19
- net TR0_TAP: now also CON5.VC1; no longer CON4.VC1
- net TR1_TAP: now also CON5.VC2; no longer CON4.VC2
- net TR2_TAP: now also CON5.VC3; no longer CON4.VC3
- net TR3_TAP: now also CON5.VC4; no longer CON4.VC4
- net TXO_N: now also CON5.TD1-, R14.2; no longer CON4.TD1-, R22.2
- net TXO_P: now also CON5.TD1+, R13.2; no longer CON4.TD1+, R21.2
- net USB0_N: now also CON3.DN1, CON3.DN2, D1.I/O_2; no longer CON5.DN1, CON5.DN2, D2.I/O_2
- net USB0_P: now also CON3.DP1, CON3.DP2, D1.I/O_1; no longer CON5.DP1, CON5.DP2, D2.I/O_1
- net USB1_N: now also CON1.D-, D2.I/O_3; no longer CON6.D-, D1.I/O_3
- net USB1_P: now also CON1.D+, D2.I/O_4; no longer CON6.D+, D1.I/O_4
- net USB2_N: now also D2.I/O_1; no longer D1.I/O_1
- net USB2_P: now also D2.I/O_2; no longer D1.I/O_2
- net VCC: now also C10.2, C15.2, CON5.A_GREEN, CON5.A_YELLOW, CON6.VCC, D3.A, J4.1, J4.17, R17.2, R19.2, R3.2, R4.1, R5.1, TP3.TP; no longer C11.2, C4.2, CON3.1, CON3.17, CON4.A_GREEN, CON4.A_YELLOW, D4.A, R1.2, R16.1, R3.1, R4.2, R5.2, TP2.TP, U$1.VCC
- net VUSB_IN: now also C5.2, CON3.VBUS, D1.REF, J3.2; no longer C1.2, CON5.VBUS, D2.REF, J1.2
Other:
- note added: "further ref: ST AN5121 https://e2e.ti.com/support/interface-group/interface/f/interface-forum/615308/tpd12s521-about-the-sch-for-tpd12s521"
